Commit message: feat(fortis_description): add stow-offset kinematics, motor visuals, transverse camera
Arm chain is no longer treated as co-linear. Adds the lateral 'stow offsets'
along each joint's rotation axis (local Y) that let the arm fold flat into
its stowed pose without segments intersecting. Values back-computed from CAD:
  J2 -> J3: y = -0.073 m  (chassis-right per REP-103)
  J3 -> J4: y = +0.052 m  (zigzag flip to chassis-left)
  J4 -> EE: y =  0.000 m  (~11 mm in CAD, treated as noise)

arm_link*_axis values now hold the X projection (tube length), not the
3D axis-to-axis distance. Total 3D distance = sqrt(X^2 + offset_y^2).

Tube visuals yaw to span the diagonal between successive joint axes
(atan2 of offset/axis). Motor body visuals added at each joint origin
(NEMA 23+50:1 at J2, NEMA 17+Cricket at J3, D845WP at J4) using catalog
dimensions, oriented with rotation axis along Y.

Arm camera (OAK-D Pro AF) rotated 90 deg about Z so the 97 mm long axis
lies transverse to the arm (parallel to gripper jaw opening direction).
Optical frame transform unchanged - the lens still points along link4 +X.

Link CoMs biased toward Y offset where the heavy motor mass actually sits.

arm_base_height: 0.030 -> 0.053 m, matching CAD J1-motor protrusion.

Build verified:
  colcon build --packages-select fortis_description
  xacro fortis_robot.urdf.xacro | check_urdf  (25 links, single root)
  pre-commit run --all-files                  (6/6 hooks pass)

File: src/fortis_description/urdf/fortis_arm.urdf.xacro (robot description, xacro)
@@ -55,4 +55,12 @@
       <material name="fortis_aluminum"/>
     </visual>
+    <!-- J2 motor body (NEMA 23 + 50:1 planetary) sits at top of L1, axis along Y. -->
+    <visual>
+      <origin xyz="0 0 ${j1_to_j2_axis}" rpy="0 0 0"/>
+      <geometry>
+        <box size="${j2_motor_x} ${j2_motor_y} ${j2_motor_z}"/>
+      </geometry>
+      <material name="fortis_motor_black"/>
+    </visual>
     <collision>
       <origin xyz="0 0 ${j1_to_j2_axis/2}" rpy="0 0 0"/>
@@ -85,6 +93,9 @@
   -->
   <link name="link2">
-    <visual>
-      <origin xyz="${arm_link2_axis/2} 0 0" rpy="0 0 0"/>
+    <!-- Tube spans diagonally from L2 origin (J2 axis) to (arm_link2_axis, j2_offset_y, 0) (J3 axis).
+         Yaw the box to align with that diagonal direction. -->
+    <visual>
+      <origin xyz="${arm_link2_axis/2} ${j2_offset_y/2} 0"
+              rpy="0 0 ${atan2(j2_offset_y, arm_link2_axis)}"/>
       <geometry>
         <box size="${arm_link2_tube} ${arm_tube_side} ${arm_tube_side}"/>
@@ -92,16 +103,26 @@
       <material name="fortis_carbon_fiber"/>
     </visual>
-    <collision>
-      <origin xyz="${arm_link2_axis/2} 0 0" rpy="0 0 0"/>
+    <!-- J3 motor body (NEMA 17 + Cricket) at the far end of L2, axis along Y. -->
+    <visual>
+      <origin xyz="${arm_link2_axis} ${j2_offset_y} 0" rpy="0 0 0"/>
+      <geometry>
+        <box size="${j3_motor_x} ${j3_motor_y} ${j3_motor_z}"/>
+      </geometry>
+      <material name="fortis_motor_black"/>
+    </visual>
+    <collision>
+      <origin xyz="${arm_link2_axis/2} ${j2_offset_y/2} 0"
+              rpy="0 0 ${atan2(j2_offset_y, arm_link2_axis)}"/>
       <geometry>
         <box size="${arm_link2_tube} ${arm_tube_side} ${arm_tube_side}"/>
       </geometry>
     </collision>
-    <!-- CoM at 75% toward J3: NEMA 17 + Cricket at J3 end dominates CF tube. -->
+    <!-- CoM at 75% toward J3 along the tube, and biased toward the Y offset
+         since the NEMA 17 + Cricket sit at the offset position, not on tube axis. -->
     <xacro:box_inertia m="${arm_link2_mass}"
                        x="${arm_link2_axis}"
                        y="${arm_tube_side}"
                        z="${arm_tube_side}"
-                       xyz="${arm_link2_axis*0.75} 0 0"/>
+                       xyz="${arm_link2_axis*0.75} ${j2_offset_y*0.6} 0"/>
   </link>
   <joint name="joint_j2" type="revolute">
@@ -116,6 +137,8 @@
   <!-- =================== J3: elbow pitch (revolute about Y) =================== -->
   <link name="link3">
-    <visual>
-      <origin xyz="${arm_link3_axis/2} 0 0" rpy="0 0 0"/>
+    <!-- Tube spans diagonally from L3 origin (J3 axis) to (arm_link3_axis, j3_offset_y, 0). -->
+    <visual>
+      <origin xyz="${arm_link3_axis/2} ${j3_offset_y/2} 0"
+              rpy="0 0 ${atan2(j3_offset_y, arm_link3_axis)}"/>
       <geometry>
         <box size="${arm_link3_tube} ${arm_tube_side} ${arm_tube_side}"/>
@@ -123,21 +146,32 @@
       <material name="fortis_carbon_fiber"/>
     </visual>
-    <collision>
-      <origin xyz="${arm_link3_axis/2} 0 0" rpy="0 0 0"/>
+    <!-- J4 servo (Hitec D845WP) at the far end of L3, axis along Y. -->
+    <visual>
+      <origin xyz="${arm_link3_axis} ${j3_offset_y} 0" rpy="0 0 0"/>
+      <geometry>
+        <box size="${j4_motor_x} ${j4_motor_y} ${j4_motor_z}"/>
+      </geometry>
+      <material name="fortis_motor_black"/>
+    </visual>
+    <collision>
+      <origin xyz="${arm_link3_axis/2} ${j3_offset_y/2} 0"
+              rpy="0 0 ${atan2(j3_offset_y, arm_link3_axis)}"/>
       <geometry>
         <box size="${arm_link3_tube} ${arm_tube_side} ${arm_tube_side}"/>
       </geometry>
     </collision>
-    <!-- CoM at 70% toward J4: D845WP servo at J4 end. -->
+    <!-- CoM at 70% toward J4 along the tube, biased toward Y offset where J4
+         servo sits (sign matches j3_offset_y -> flipped from j2 side). -->
     <xacro:box_inertia m="${arm_link3_mass}"
                        x="${arm_link3_axis}"
                        y="${arm_tube_side}"
                        z="${arm_tube_side}"
-                       xyz="${arm_link3_axis*0.70} 0 0"/>
+                       xyz="${arm_link3_axis*0.70} ${j3_offset_y*0.6} 0"/>
   </link>
   <joint name="joint_j3" type="revolute">
     <parent link="link2"/>
     <child  link="link3"/>
-    <origin xyz="${arm_link2_axis} 0 0" rpy="0 0 0"/>
+    <!-- Y component is the lateral stow offset along J2 rotation axis. -->
+    <origin xyz="${arm_link2_axis} ${j2_offset_y} 0" rpy="0 0 0"/>
     <axis xyz="0 1 0"/>
     <limit lower="${j3_lower}" upper="${j3_upper}"
@@ -169,5 +203,6 @@
     <parent link="link3"/>
     <child  link="link4"/>
-    <origin xyz="${arm_link3_axis} 0 0" rpy="0 0 0"/>
+    <!-- Zigzag flip: J3 offset is +Y (opposite to J2 which was -Y). -->
+    <origin xyz="${arm_link3_axis} ${j3_offset_y} 0" rpy="0 0 0"/>
     <axis xyz="0 1 0"/>
     <limit lower="${j4_lower}" upper="${j4_upper}"
@@ -203,5 +238,5 @@
     <parent link="link4"/>
     <child  link="ee"/>
-    <origin xyz="${arm_link4_axis} 0 0" rpy="0 0 0"/>
+    <origin xyz="${arm_link4_axis} ${j4_offset_y} 0" rpy="0 0 0"/>
   </joint>
   <!-- =================== gripper jaws =================== -->
@@ -272,7 +307,13 @@
   </joint>
   <!-- =================== arm camera (OAK-D Pro AF) =================== -->
+  <!--
+    Camera body rotated 90 deg about Z so the 97 mm long dimension lies along
+    link4's local +Y (transverse to the arm tube, parallel to the gripper
+    jaw-opening axis). Lens still points along link4's +X (arm-forward), so
+    the optical frame transform downstream is unchanged.
+  -->
   <link name="arm_camera_link">
     <visual>
-      <origin xyz="0 0 0" rpy="0 0 0"/>
+      <origin xyz="0 0 0" rpy="0 0 ${pi/2}"/>
       <geometry>
         <box size="${oak_pro_x} ${oak_pro_y} ${oak_pro_z}"/>
@@ -281,5 +322,5 @@
     </visual>
     <collision>
-      <origin xyz="0 0 0" rpy="0 0 0"/>
+      <origin xyz="0 0 0" rpy="0 0 ${pi/2}"/>
       <geometry>
         <box size="${oak_pro_x} ${oak_pro_y} ${oak_pro_z}"/>
@@ -289,5 +330,6 @@
                        x="${oak_pro_x}"
                        y="${oak_pro_y}"
-                       z="${oak_pro_z}"/>
+                       z="${oak_pro_z}"
+                       rpy="0 0 ${pi/2}"/>
   </link>
   <!--

File: src/fortis_description/urdf/fortis_constants.xacro (robot description, xacro)
@@ -38,15 +38,52 @@
     The difference per segment is split evenly when placing the tube visual.
   -->
+  <!--
+    Axis-to-axis X-projections (along the tube), NOT diagonal distances.
+    The arm has lateral stow offsets at each joint (j*_offset_y below) so the
+    full 3D distance from one joint axis to the next is sqrt(axis^2 + offset_y^2).
+    These values were back-computed from CAD-extracted joint origins.
+  -->
   <xacro:property name="j1_to_j2_axis"   value="0.091"/>  <!--  3.59 in -->
-  <xacro:property name="arm_link2_axis"  value="0.411"/>  <!-- 16.16 in, J2 axis to J3 axis -->
-  <xacro:property name="arm_link3_axis"  value="0.300"/>  <!-- 11.82 in, J3 axis to J4 axis -->
-  <xacro:property name="arm_link4_axis"  value="0.068"/>  <!--  2.68 in, J4 axis to EE attach -->
+  <xacro:property name="arm_link2_axis"  value="0.404"/>  <!-- 15.91 in, J2->J3 X-projection (3D dist 0.411) -->
+  <xacro:property name="arm_link3_axis"  value="0.295"/>  <!-- 11.61 in, J3->J4 X-projection (3D dist 0.300) -->
+  <xacro:property name="arm_link4_axis"  value="0.060"/>  <!--  2.36 in, J4 axis to EE attach (CAD verified) -->
   <xacro:property name="ee_to_gripper"   value="0.030"/>  <!--  1.20 in, EE attach to gripper base -->
+  <!--
+    Lateral "stow" offsets at each joint along the joint's rotation axis (local Y).
+    This is what lets L2's plane of motion sit alongside L1's plane instead of
+    on top of it, so the arm can fold flat. Sign convention follows REP-103
+    (+Y = chassis left, -Y = chassis right). Per FORTIS spec:
+      J2 motor mounts on chassis-right side -> j2_offset_y is NEGATIVE
+      J3 motor mounts opposite (chassis-left) -> j3_offset_y is POSITIVE
+      J4 mounts same side as J3 (~negligible)  -> j4_offset_y ~ 0
+  -->
+  <xacro:property name="j2_offset_y"     value="-0.073"/> <!-- L2 to J3 axis, CAD-extracted -->
+  <xacro:property name="j3_offset_y"     value="+0.052"/> <!-- L3 to J4 axis, CAD-extracted -->
+  <xacro:property name="j4_offset_y"     value="0.000"/>  <!-- L4 to EE attach; 11 mm in CAD, treated as noise -->
+  <xacro:property name="ee_offset_y"     value="0.000"/>  <!-- EE attach to gripper base -->
   <xacro:property name="arm_link2_tube"  value="0.360"/>  <!-- 14.17 in, j2_link CF tube -->
   <xacro:property name="arm_link3_tube"  value="0.208"/>  <!--  8.18 in, j3_link CF tube -->
   <xacro:property name="arm_link4_tube"  value="0.038"/>  <!--  1.50 in, j4_link -->
   <xacro:property name="arm_tube_side"   value="0.0287"/> <!--  1.128 in, square CF tube outer -->
-  <!-- Arm base (J1 motor body) sits on chassis, joint_j1 axis at its top. -->
-  <xacro:property name="arm_base_height" value="0.030"/>  <!-- ~NEMA 17 body height -->
+  <!--
+    Arm base (J1 motor body) protrudes above chassis top. The motor body extends
+    DOWN into the chassis; the rotation axis sits at the top of the housing.
+    Value matches CAD-extracted J1 axis height above chassis-arm interface plane.
+  -->
+  <xacro:property name="arm_base_height" value="0.053"/>  <!-- CAD verified -->
+  <!--
+    Motor body visual primitives. Catalog dimensions from data sheets; used as
+    cosmetic boxes at each joint origin so the arm renders as a continuous
+    object rather than floating tube segments.
+  -->
+  <xacro:property name="j2_motor_x"      value="0.057"/>  <!-- NEMA 23 cross-section -->
+  <xacro:property name="j2_motor_y"      value="0.120"/>  <!-- NEMA 23 + 50:1 planetary, total length along axis -->
+  <xacro:property name="j2_motor_z"      value="0.057"/>
+  <xacro:property name="j3_motor_x"      value="0.042"/>  <!-- NEMA 17 cross-section -->
+  <xacro:property name="j3_motor_y"      value="0.080"/>  <!-- NEMA 17 + Cricket gearbox, total length along axis -->
+  <xacro:property name="j3_motor_z"      value="0.042"/>
+  <xacro:property name="j4_motor_x"      value="0.040"/>  <!-- Hitec D845WP servo -->
+  <xacro:property name="j4_motor_y"      value="0.038"/>
+  <xacro:property name="j4_motor_z"      value="0.020"/>
   <!--
     Composite link masses. Each "linkN" rotates with jointN, so the inertia must
