Commit message: fix(kinematics): wheelbase/track from measured contact spans
LEN_X 0.176->0.174625 (13.75 in front-back /2), LEN_Y 0.125->0.12065 (9.5 in left-right /2). URDF wheel_x/y_offset updated to match (keeps test_kinematics_urdf_sync passing). Measured 2026-06-07.

File: src/fortis_description/urdf/fortis_constants.xacro (robot description, xacro)
@@ -18,7 +18,7 @@
   <xacro:property name="wheel_width"     value="0.051"/>  <!-- 2.000 in -->
   <xacro:property name="wheel_mass"      value="1.0"/>    <!-- ~1 kg per wheel -->
-  <!-- Wheel center positions from chassis center (extracted from CAD) -->
-  <xacro:property name="wheel_x_offset"  value="0.176"/>  <!-- 6.93 in, half longitudinal spread -->
-  <xacro:property name="wheel_y_offset"  value="0.125"/>  <!-- 4.92 in, half lateral spread -->
+  <!-- Wheel center positions from chassis center (measured contact spans 2026-06-07) -->
+  <xacro:property name="wheel_x_offset"  value="0.174625"/>  <!-- half of 13.75 in front-back span -->
+  <xacro:property name="wheel_y_offset"  value="0.12065"/>  <!-- half of 9.5 in left-right span -->
   <xacro:property name="wheel_z"         value="${wheel_radius}"/>  <!-- wheel center at axle height -->
   <!-- X-config: each wheel rotated 45 deg about Z so its rolling axis is diagonal -->
